Commit message: act: Complete RTAB-Map project Add a new mapping.launch file Add a new robot urdf file with simulated Kinect sensor

File: my_robot/urdf/my_robot.xacro (robot description, xacro)
@@ -150,4 +150,11 @@
 		<parent link="chassis"/>
 	</joint>
+	<joint name="camera_optical_joint" type="fixed">
+		<origin xyz="0 0 0" rpy="-1.5707 0 -1.5707"/>
+		<parent link="camera"/>
+		<child link="camera_link_optical"/>
+	</joint>
+	<link name="camera_link_optical">
+		</link>
 	<!-- LIDAR = Hokuyo Sensor -->
 	<link name="hokuyo">
